File: code/hw_lower_v1/hw_lower_v1/hw_lower_v1.kicad_sch (KiCad schematic)
At the start: 35 parts, among them J1 Conn_01x24_Socket, J2 Conn_01x03_Pin, J3 Conn_01x03_Pin, Q1 BS108, U1 LM397, U2 DRV8837C, U3 SST25VF080B-50-4x-S2Ax

Commit message: started full lower pcb version
Parts:
- removed D1: D, symbol Device:D
- removed J2, J3: Conn_01x03_Pin, symbol Connector:Conn_01x03_Pin
- removed K1: ~, symbol hw_lower_v1:Panasonic_HE-R_2
- removed Q1: BS108, Package_TO_SOT_THT:TO-92_Inline, symbol Transistor_FET:BS108
- removed R1: R, symbol Device:R
- removed R9: R?, symbol Device:R
Connections:
- net Earth renamed GND
Other:
- added sheet AC (AC.kicad_sch)
- note added: "GFCI CAL"
- note added: "GFCI FAULT"
- note removed: "12V 5V 3V3 GND -12V"
- note removed: "AC + DC FAULT"
- note removed: "DC FAULT"
- note removed: "GFCI"
- note removed: "L"
- note removed: "N"
- note removed: "ONLY FOR GFCI ~100mA"
- note removed: "PE"
- note removed: "POWER L AC N"
- note removed: "POWER_MEASUREMENT"
- note removed: "SOLDER SCREW HOLES"
- moved on the sheet: C1, C2, C3, D2, H1, H2, H3, H4, H5, H6, J1, R10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
