File: code/hw_upper_v1/hw_upper_v1/hw_upper_v1.kicad_pcb (KiCad board)
At the start: 2 copper layers, 102 x 49 mm, 11 parts, among them J1 Conn_02x20_Odd_Even

Commit message: have one project part library
Parts:
- moved FID2 6.95 mm to (97.0, 112.0)
- moved FID5 6.95 mm to (97.0, 112.0)
- moved FID1 2.00 mm to (103.0, 75.5)
- moved FID3 1.12 mm to (193.0, 82.0)
- moved FID6 1.12 mm to (193.0, 82.0)
Other:
- outline, holes or cut-outs redrawn
- board text added: "fillet: 3.5mm"
Changed lines of the file:
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@@
 	(footprint "Fiducial:Fiducial_1mm_Mask3mm"
 		(layer "F.Cu")
-		(at 103 77.5)
+		(at 103 75.5)
 		(descr "Circular Fiducial, 1mm bare copper, 3mm soldermask opening (recommended)")
 		(tags "fiducial")
@@
 	(footprint "Fiducial:Fiducial_1mm_Mask3mm"
 		(layer "F.Cu")
-		(at 103 115.5)
+		(at 97 112)
 		(descr "Circular Fiducial, 1mm bare copper, 3mm soldermask opening (recommended)")
 		(tags "fiducial")
@@
 	(footprint "Fiducial:Fiducial_1mm_Mask3mm"
 		(layer "F.Cu")
-		(at 192.5 83)
+		(at 193 82)
 		(descr "Circular Fiducial, 1mm bare copper, 3mm soldermask opening (recommended)")
 		(tags "fiducial")
@@
 	(footprint "Fiducial:Fiducial_1mm_Mask3mm"
 		(layer "B.Cu")
-		(at 192.5 83 180)
+		(at 193 82 180)
 		(descr "Circular Fiducial, 1mm bare copper, 3mm soldermask opening (recommended)")
 		(tags "fiducial")
@@
 	(footprint "Fiducial:Fiducial_1mm_Mask3mm"
 		(layer "B.Cu")
-		(at 103 115.5 180)
+		(at 97 112 180)
 		(descr "Circular Fiducial, 1mm bare copper, 3mm soldermask opening (recommended)")
 		(tags "fiducial")
@@
 		(layer "Dwgs.User")
 	)
-	(gr_rect
-		(start 94 72.5)
-		(end 196 121.5)
+	(gr_arc
+		(start 196 118)
+		(mid 194.974874 120.474874)
+		(end 192.5 121.5)
+		(stroke
+			(width 0.05)
+			(type default)
+		)
+		(layer "Edge.Cuts")
+	)
+	(gr_line
+		(start 192.5 121.5)
+		(end 97.5 121.5)
+		(stroke
+			(width 0.05)
+			(type default)
+		)
+		(layer "Edge.Cuts")
+	)
+	(gr_arc
+		(start 94 76)
+		(mid 95.025126 73.525126)
+		(end 97.5 72.5)
+		(stroke
+			(width 0.05)
+			(type default)
+		)
+		(layer "Edge.Cuts")
+	)
+	(gr_line
+		(start 97.5 72.5)
+		(end 192.5 72.5)
+		(stroke
+			(width 0.05)
+			(type default)
+		)
+		(layer "Edge.Cuts")
+	)
+	(gr_arc
+		(start 97.5 121.5)
+		(mid 95.025126 120.474874)
+		(end 94 118)
+		(stroke
+			(width 0.05)
+			(type default)
+		)
+		(layer "Edge.Cuts")
+	)
+	(gr_arc
+		(start 192.5 72.5)
+		(mid 194.974874 73.525126)
+		(end 196 76)
+		(stroke
+			(width 0.05)
+			(type default)
+		)
+		(layer "Edge.Cuts")
+	)
+	(gr_line
+		(start 196 76)
+		(end 196 118)
+		(stroke
+			(width 0.05)
+			(type default)
+		)
+		(layer "Edge.Cuts")
+	)
+	(gr_line
+		(start 94 118)
+		(end 94 76)
 		(stroke
 			(width 0.05)
 			(type default)
 		)
-		(fill none)
 		(layer "Edge.Cuts")
 	)
@@
 		)
 	)
+	(gr_text "fillet: 3.5mm"
+		(at 92 124.5 0)
+		(layer "User.7")
+		(effects
+			(font
+				(size 1.5 1.5)
+				(thickness 0.3)
+				(bold yes)
+			)
+			(justify left bottom)
+		)
+	)

Commit message: before the final route
Parts:
- added H5: MountingHole, MountingHole:MountingHole_3.2mm_M3_Pad, F.Cu at (192.5, 118.0)
- moved J1 1.11 mm to (184.9, 115.5)
Routing:
- net unconnected-(J1-Pin_15-Pad15): track 0.00 -> 9.23 mm
- net unconnected-(J1-Pin_25-Pad25): track 0.00 -> 6.50 mm
- net unconnected-(J1-Pin_11-Pad11): track 0.00 -> 4.69 mm
- net unconnected-(J1-Pin_39-Pad39): track 0.00 -> 3.11 mm
- net unconnected-(J1-Pin_33-Pad33): track 0.00 -> 3.06 mm
- net unconnected-(J1-Pin_17-Pad17): track 0.00 -> 3.03 mm
- net unconnected-(J1-Pin_27-Pad27): track 0.00 -> 2.93 mm
Changed lines of the file:
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@@
 	(footprint "Connector_PinHeader_2.54mm:PinHeader_2x20_P2.54mm_Vertical"
 		(layer "F.Cu")
-		(at 185.7 116.21 -90)
+		(at 184.88 115.46 -90)
 		(descr "Through hole straight pin header, 2x20, 2.54mm pitch, double rows")
 		(tags "Through hole pin header THT 2x20 2.54mm double row")
@@
 		)
 		(fp_text user "${REFERENCE}"
-			(at 1.27 24.13 360)
+			(at 1.27 24.13 0)
 			(layer "F.Fab")
 			(effects
@@
 	(footprint "MountingHole:MountingHole_3.2mm_M3_Pad"
 		(layer "F.Cu")
+		(at 192.5 118 -90)
+		(descr "Mounting Hole 3.2mm, M3")
+		(tags "mounting hole 3.2mm m3")
+		(property "Reference" "H5"
+			(at 0 -4.2 -90)
+			(layer "F.SilkS")
+			(hide yes)
+			(effects
+				(font
+					(size 1 1)
+					(thickness 0.15)
+				)
+			)
+		)
+		(property "Value" "MountingHole"
+			(at 0 4.2 -90)
+			(layer "F.Fab")
+			(effects
+				(font
+					(size 1 1)
+					(thickness 0.15)
+				)
+			)
+		)
+		(property "Footprint" "MountingHole:MountingHole_3.2mm_M3_Pad"
+			(at 0 0 -90)
+			(unlocked yes)
+			(layer "F.Fab")
+			(hide yes)
+			(effects
+				(font
+					(size 1.27 1.27)
+					(thickness 0.15)
+				)
+			)
+		)
+		(property "Datasheet" ""
+			(at 0 0 -90)
+			(unlocked yes)
+			(layer "F.Fab")
+			(hide yes)
+			(effects
+				(font
+					(size 1.27 1.27)
+					(thickness 0.15)
+				)
+			)
+		)
+		(property "Description" "Mounting Hole without connection"
+			(at 0 0 -90)
+			(unlocked yes)
+			(layer "F.Fab")
+			(hide yes)
+			(effects
+				(font
+					(size 1.27 1.27)
+					(thickness 0.15)
+				)
+			)
+		)
+		(property "Name" ""
+			(at 0 0 -90)
+			(unlocked yes)
+			(layer "F.Fab")
+			(hide yes)
+			(effects
+				(font
+					(size 1 1)
+					(thickness 0.15)
+				)
+			)
+		)
+		(attr exclude_from_pos_files exclude_from_bom)
+		(fp_circle
+			(center 0 0)
+			(end 3.2 0)
+			(stroke
+				(width 0.15)
+				(type solid)
+			)
+			(fill none)
+			(layer "Cmts.User")
+		)
+		(fp_circle
+			(center 0 0)
+			(end 3.45 0)
+			(stroke
+				(width 0.05)
+				(type solid)
+			)
+			(fill none)
+			(layer "F.CrtYd")
+		)
+		(fp_text user "${REFERENCE}"
+			(at 0 0 -90)
+			(layer "F.Fab")
+			(effects
+				(font
+					(size 1 1)
+					(thickness 0.15)
+				)
+			)
+		)
+		(pad "1" thru_hole circle
+			(at 0 0 270)
+			(size 6.4 6.4)
+			(drill 3.2)
+			(layers "*.Cu" "*.Mask")
+			(remove_unused_layers no)
+		)
+	)
+	(footprint "MountingHole:MountingHole_3.2mm_M3_Pad"
+		(layer "F.Cu")
 		(at 97.5 76)
 		(descr "Mounting Hole 3.2mm, M3")
@@
 		(layer "Edge.Cuts")
 	)
+	(gr_arc
+		(start 196 118)
+		(mid 194.974874 120.474874)
+		(end 192.5 121.5)
+		(stroke
+			(width 0.05)
+			(type default)
+		)
+		(layer "Edge.Cuts")
+	)
 	(gr_line
 		(start 192.5 121.5)
@@
 		)
 	)
+	(segment
+		(start 173.43 112.4)
+		(end 171.91 112.4)
+		(width 0.2)
+		(layer "F.Cu")
+		(net 1)
+	)
+	(segment
+		(start 172.18 112.67)
+		(end 172.18 115.46)
+		(width 0.2)
+		(layer "F.Cu")
+		(net 1)
+	)
+	(segment
+		(start 171.91 112.4)
+		(end 172.18 112.67)
+		(width 0.2)
+		(layer "F.Cu")
+		(net 1)
+	)
+	(segment
+		(start 144.38 115.32)
+		(end 144.24 115.46)
+		(width 0.2)
+		(layer "F.Cu")
+		(net 7)
+	)
+	(segment
+		(start 144.38 112.46)
+		(end 144.38 115.32)
+		(width 0.2)
+		(layer "F.Cu")
+		(net 7)
+	)
+	(segment
+		(start 139.13 118)
+		(end 139.16 118)
+		(width 0.2)
+		(layer "B.Cu")
+		(net 10)
+	)
+	(segment
+		(start 164.56 115.46)
+		(end 162.42 113.32)
+		(width 0.2)
+		(layer "B.Cu")
+		(net 11)
+	)
+	(segment
+		(start 136.68 115.4)
+		(end 136.62 115.46)
+		(width 0.2)
+		(layer "F.Cu")
+		(net 15)
+	)
+	(segment
+		(start 136.68 112.375)
+		(end 136.68 115.4)
+		(width 0.2)
+		(layer "F.Cu")
+		(net 15)
+	)
+	(segment
+		(start 151.86 112.53)
+		(end 151.86 115.46)
+		(width 0.2)
+		(layer "B.Cu")
+		(net 17)
+	)
+	(segment
+		(start 167.1 112.285)
+		(end 167.1 115.46)
+		(width 0.2)
+		(layer "F.Cu")
+		(net 27)
+	)
+	(segment
+		(start 162.82 111.18)
+		(end 167.1 115.46)
+		(width 0.2)
+		(layer "B.Cu")
+		(net 27)
+	)
+	(segment
+		(start 154.38 112.46)
+		(end 154.38 115.44)
+		(width 0.2)
+		(layer "F.Cu")
+		(net 30)
+	)
+	(segment
+		(start 154.38 115.44)
+		(end 154.4 115.46)
+		(width 0.2)
+		(layer "F.Cu")
+		(net 30)
+	)
+	(segment
+		(start 154.4 111.97)
+		(end 154.4 115.46)
+		(width 0.2)
+		(layer "B.Cu")
+		(net 30)
+	)
+	(segment
+		(start 161.88 115.32)
+		(end 162.02 115.46)
+		(width 0.2)
+		(layer "F.Cu")
+		(net 38)
+	)
 	(group ""

Commit message: moved stuff around a little bit, will optimise the number of components now
Parts:
- removed H1, H2, H3, H4, H5: MountingHole, MountingHole:MountingHole_3.2mm_M3_Pad
- moved J1 396.9 mm to (492.5, -135.2)
- moved FID2 393.3 mm to (441.8, -77.2)
- moved FID5 393.3 mm to (441.8, -77.2)
- moved FID4 385.6 mm to (461.0, -48.5)
- moved FID1 378.1 mm to (456.5, -58.7)
- moved FID3 294.1 mm to (445.8, -68.5)
- moved FID6 294.1 mm to (445.8, -68.5)
Routing:
- net unconnected-(J1-Pin_15-Pad15): track 9.23 -> 0.00 mm
- net unconnected-(J1-Pin_25-Pad25): track 6.50 -> 0.00 mm
- net unconnected-(J1-Pin_11-Pad11): track 4.69 -> 0.00 mm
- net unconnected-(J1-Pin_39-Pad39): track 3.11 -> 0.00 mm
- net unconnected-(J1-Pin_33-Pad33): track 3.06 -> 0.00 mm
- net unconnected-(J1-Pin_17-Pad17): track 3.03 -> 0.00 mm
- net unconnected-(J1-Pin_27-Pad27): track 2.93 -> 0.00 mm
Other:
- board text removed: "R2"
- board text removed: "R4"
- board text removed: "R6"
