File: code/hw_lower_v2/hw_lower_v2/hw_lower_v2.kicad_pcb (KiCad board)
At the start: 4 copper layers, 102 x 104.8 mm, 115 parts, among them J1 Screw_Terminal_01x01, J14 Conn_01x02, J2 Screw_Terminal_01x01, J3 Screw_Terminal_01x01, J4 Screw_Terminal_01x01, J5 Screw_Terminal_01x01, J6 Screw_Terminal_01x01, J7 Conn_01x06_Pin, J8 Conn_02x20_Odd_Even, K1 AHES4191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

Commit message: simplify component values
Parts:
- R14, R17, R18, R19, R29, R33: value 1K -> 510R
- R15: value 100k -> 200K 1%
- R2, R35, R36, R4, R6: value 100K -> 10K
- R24: value 56k -> 10K
- R26: value 100k -> 20K
- R31: value 200k 1% -> 200K 1%
- R37: value 160R -> 120R
Changed lines of the file:
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@@
 			)
 		)
-		(property "Value" "1K"
+		(property "Value" "510R"
 			(at 0 1.43 0)
 			(layer "F.Fab")
@@
 			)
 		)
-		(property "LCSC" "C21190"
+		(property "LCSC" "C23193"
 			(at 0 0 0)
 			(unlocked yes)
@@
 			)
 		)
-		(property "Value" "100k"
+		(property "Value" "200K 1%"
 			(at 0 1.43 0)
 			(layer "F.Fab")
@@
 			)
 		)
-		(property "LCSC" "C25804"
+		(property "LCSC" "C2989567"
 			(at 0 0 180)
 			(unlocked yes)
@@
 			)
 		)
-		(property "Value" "100K"
+		(property "Value" "10K"
 			(at 0 1.43 0)
 			(layer "F.Fab")
@@
 			)
 		)
-		(property "LCSC" "C25803"
+		(property "LCSC" "C25804"
 			(at 0 0 0)
 			(unlocked yes)
@@
 			)
 		)
-		(property "Value" "1K"
+		(property "Value" "510R"
 			(at 0 1.43 0)
 			(layer "F.Fab")
@@
 			)
 		)
-		(property "LCSC" "C21190"
+		(property "LCSC" "C23193"
 			(at 0 0 180)
 			(unlocked yes)
@@
 			)
 		)
-		(property "Value" "1K"
+		(property "Value" "510R"
 			(at 0 1.43 0)
 			(layer "F.Fab")
@@
 			)
 		)
-		(property "LCSC" "C21190"
+		(property "LCSC" "C23193"
 			(at 0 0 0)
 			(unlocked yes)
@@
 			)
 		)
-		(property "Value" "200k 1%"
+		(property "Value" "200K 1%"
 			(at 0 1.43 90)
 			(layer "F.Fab")
@@
 			)
 		)
-		(property "Value" "100K"
+		(property "Value" "10K"
 			(at 0 1.43 90)
 			(layer "F.Fab")
@@
 			)
 		)
-		(property "LCSC" "C25803"
+		(property "LCSC" "C25804"
 			(at 0 0 -90)
 			(unlocked yes)
@@
 			)
 		)
-		(property "Value" "100K"
+		(property "Value" "10K"
 			(at 0 1.43 90)
 			(layer "F.Fab")
@@
 			)
 		)
-		(property "LCSC" "C25803"
+		(property "LCSC" "C25804"
 			(at 0 0 -90)
 			(unlocked yes)
@@
 			)
 		)
-		(property "Value" "1K"
+		(property "Value" "510R"
 			(at 0 1.43 0)
 			(layer "F.Fab")
@@
 			)
 		)
-		(property "LCSC" "C21190"
+		(property "LCSC" "C23193"
 			(at 0 0 180)
 			(unlocked yes)
@@
 			)
 		)
-		(property "Value" "1K"
+		(property "Value" "510R"
 			(at 0 1.43 0)
 			(layer "F.Fab")
@@
 			)
 		)
-		(property "LCSC" "C21190"
+		(property "LCSC" "C23193"
 			(at 0 0 180)
 			(unlocked yes)
@@
 			)
 		)
-		(property "Value" "160R"
+		(property "Value" "120R"
 			(at 0 1.43 0)
 			(layer "F.Fab")
@@
 			)
 		)
-		(property "LCSC" "C22814"
+		(property "LCSC" "C125925"
 			(at 0 0 0)
 			(unlocked yes)
@@
 			)
 		)
-		(property "Value" "100K"
+		(property "Value" "10K"
 			(at 0 1.43 0)
 			(layer "F.Fab")
@@
 			)
 		)
-		(property "LCSC" "C25803"
+		(property "LCSC" "C25804"
 			(at 0 0 180)
 			(unlocked yes)
@@
 			)
 		)
-		(property "Value" "100k"
+		(property "Value" "20K"
 			(at 0 1.43 90)
 			(layer "F.Fab")
@@
 			)
 		)
-		(property "LCSC" "C25804"
+		(property "LCSC" "C706407"
 			(at 0 0 -90)
 			(unlocked yes)
@@
 			)
 		)
-		(property "Value" "56k"
+		(property "Value" "10K"
 			(at 0 1.43 90)
 			(layer "F.Fab")
@@
 			)
 		)
-		(property "LCSC" "C5250755"
+		(property "LCSC" "C25804"
 			(at 0 0 90)
 			(unlocked yes)
@@
 			)
 		)
-		(property "Value" "1K"
+		(property "Value" "510R"
 			(at 0 1.43 90)
 			(layer "F.Fab")
@@
 			)
 		)
-		(property "LCSC" "C21190"
+		(property "LCSC" "C23193"
 			(at 0 0 -90)
 			(unlocked yes)
@@
 			)
 		)
-		(property "Value" "100K"
+		(property "Value" "10K"
 			(at 0 1.43 90)
 			(layer "F.Fab")
@@
 			)
 		)
-		(property "LCSC" "C25803"
+		(property "LCSC" "C25804"
 			(at 0 0 -90)
 			(unlocked yes)
