File: code/hw_lower_v2/hw_lower_v2/AC.kicad_sch (KiCad schematic)
At the start: 38 parts, among them K1 AHES4191, Q1 BSS138, Q2 BSS138, Q3 BSS138, T1 TS3193-2C 2mA/2mA, U1 BRCS02C, U2 BL0942

Commit message: wip
Parts:
- removed Q2, Q3: BSS138, Package_TO_SOT_SMD:SOT-23, symbol Transistor_FET:BSS138
- removed R21, R22, R23, R45: 10K, Resistor_SMD:R_0603_1608Metric, symbol Device:R
- C2: LCSC C72485 -> C86602
Connections:
- net +3.3V: now also R20.2
- net +5V: no longer R20.2
- net GFCI_CALIBRATE: now also R20.1, U1.5 (Cal)
- net GFCI_TEST: now also U1.6 (TEST)
Other:
- note added: "UART- DNP SPI - 0 Ohm"
- moved on the sheet: R20, R24, R26
