File: code/hw_lower_v2/hw_lower_v2/hw_lower_v2.kicad_sch (KiCad schematic)
At the start: 26 parts, among them J1 Screw_Terminal_01x01, J2 Screw_Terminal_01x01, J3 Screw_Terminal_01x01, J4 Screw_Terminal_01x01, J5 Screw_Terminal_01x01, J6 Screw_Terminal_01x01, J7 Conn_01x06_Pin, J8 Conn_02x20_Odd_Even

Commit message: wip
Other:
- note added: "- more resistors in the Vac string - check gfci cal with just a pullup -"
Changed lines of the file:
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@@
+		)
+	)
+	(text "- more resistors in the Vac string\n- check gfci cal with just a pullup\n- "
+		(exclude_from_sim no)
+		(at 158.75 25.146 0)
+		(effects
+			(font
+				(size 1.27 1.27)
+			)
+			(justify left)
 		)
 	)
